File: midi_switcher_dpdt/midi-switcher-dpdt.brd (EAGLE design)
At the start: 123.1 x 54.4 mm, 106 parts, among them IC1 6N138, IC2 PIC16F1825SO14, IC4 REG1117

Commit message: first layout dpdt
Routing:
- net OUT1: track 75.1 -> 69.8 mm
- net SWITCH: track 38.9 -> 44.0 mm
- net ACT_LED: track 22.6 -> 24.4 mm, vias 3 -> 2
- net +9V: track 188.3 -> 189.8 mm
- net OUT8: track 62.4 -> 61.2 mm
- net OUT4: track 13.4 -> 12.3 mm
- net MIDI_IN: vias 3 -> 2

Commit message: Update midi-switcher-dpdt.brd
Parts:
- flipped NC1 to the top
Routing:
- net +5V: track 95.2 -> 85.1 mm
- net +9V: track 189.8 -> 190.6 mm
- net N$65: track 15.9 -> 15.3 mm
- added copper zone on layer 1, net AGND
- added copper zone on layer 16, net GND
Other:
- board text added: "A"
- board text added: "B"
- board text added: "C"
- board text added: "D"
- board text added: "E"
- board text added: "F"
- board text added: "G"
- board text added: "H"

Commit message: dsf
Parts:
- removed R23, R24, R25: (no value), rcl:R0805
- removed U$10: 0805DIODE, jasons_stuff:0805DIODE
- added D2: MBR0520LT, diode:SOD123
- added R19, R7, R9: (no value), rcl:R0805
- D3: value MBR0520LT -> 0805DIODE; device diode:SOD123 -> jasons_stuff:0805DIODE
- moved R20 92.5 mm to (98.9, 39.7)
- moved R8 87.5 mm to (8.90, 39.7)
- moved D3 85.9 mm to (15.9, 39.7)
- moved R17 72.5 mm to (81.4, 39.7)
- moved R22 63.6 mm to (113.9, 39.7), turned to 270 degrees
- moved R18 62.5 mm to (83.9, 39.7)
- moved R21 60.7 mm to (111.4, 39.7), turned to 270 degrees
- moved R3 60.7 mm to (51.5, 49.5), turned to 180 degrees
- moved R10 57.5 mm to (23.9, 39.7)
- moved R15 42.5 mm to (66.4, 39.7)
- moved R6 35.4 mm to (82.0, 55.0)
- moved R5 32.7 mm to (70.0, 55.0)
- moved R4 32.6 mm to (51.5, 43.5), turned to 0 degrees
- moved R16 32.5 mm to (68.9, 39.7)
- moved R12 27.5 mm to (38.9, 39.7)
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- renumbered Q9 to TR1, T1 to TR2, T2 to TR3, T3 to TR4, T4 to TR5, T5 to TR6, T6 to TR7, T7 to TR8, T8 to TR9, U$11 to D4, U$12 to D5, U$13 to D6, U$14 to D7, U$15 to D8, U$16 to D9, U$17 to D10
Connections:
- net +5V: now also R2.2; no longer R22.2
- net +9V: now also D2.C, D3.A; no longer D3.C, U$10.A
- net GND: now also R3.1, R5.2, R6.2; no longer R21.1, R24.2, R25.2
- net MIDI_IN: now also R2.1; no longer R22.1
- net N$12: now also R10.2; no longer R15.2
- net N$15: now also R12.2; no longer R13.2
- net N$16: now also R4.2; no longer R23.2
- net N$18: now also R4.1; no longer R23.1
- net N$20: now also R14.2; no longer R11.2
- net N$21: now also D2.A; no longer D3.A
- net N$24: now also R11.2; no longer R16.2
- net N$28: now also R6.1; no longer R24.1
- net N$33: now also R13.2; no longer R14.2
- net N$35: now also R15.2; no longer R12.2
- net N$36: now also R17.2; no longer R10.2
- net N$37: now also R19.2; no longer R8.2
- net N$38: now also R21.2; no longer R3.2
- net N$4: now also R3.2; no longer R21.2
- net N$5: now also R5.1; no longer R25.1
- net N$57: now also R16.2; no longer R2.2
- net N$6: now also R7.2; no longer R20.2
- net N$60: now also R18.2; no longer R4.2
- net N$63: now also R20.2; no longer R5.2
- net N$66: now also R22.2; no longer R6.2
- net N$7: now also R9.2; no longer R18.2
- net N$8: now also D3.C; no longer U$10.C
- net N$9: now also R8.2; no longer R17.2
- net OUT1: now also R7.1, R8.1; no longer R17.1, R20.1
- net OUT2: now also R10.1, R9.1; no longer R15.1, R18.1
- net OUT3: now also R11.1, R12.1; no longer R13.1, R16.1
- net OUT4: now also R13.1; no longer R11.1
- net OUT5: now also R15.1, R16.1; no longer R12.1, R2.1
- net OUT6: now also R17.1, R18.1; no longer R10.1, R4.1
- net OUT7: now also R19.1, R20.1; no longer R5.1, R8.1
- net OUT8: now also R21.1, R22.1; no longer R3.1, R6.1
Other:
- board text added: "PWR POL"
