File: midi_switcher_dpdt/midi-switcher-dpdt.sch (EAGLE design)
At the start: 106 parts, among them IC1 6N138, IC2 PIC16F1825SO14, IC4 REG1117

Commit message: dsf
Parts:
- removed R23, R24, R25: (no value), rcl:R-EU_R0805
- removed U$10: 0805DIODE, jasons_stuff:0805DIODE
- added D2: MBR0520LT, diode:MBR0520LT
- added R19, R7, R9: (no value), rcl:R-EU_R0805
- D3: value MBR0520LT -> 0805DIODE; device diode:MBR0520LT -> jasons_stuff:0805DIODE
- renumbered Q9 to TR1, T1 to TR2, T2 to TR3, T3 to TR4, T4 to TR5, T5 to TR6, T6 to TR7, T7 to TR8, T8 to TR9, U$11 to D4, U$12 to D5, U$13 to D6, U$14 to D7, U$15 to D8, U$16 to D9, U$17 to D10
Connections:
- net +5V: now also R2.2; no longer R22.2
- net +9V: now also D2.C, D3.P$2; no longer D3.C, U$10.P$2
- net GND: now also R3.1, R5.2, R6.2; no longer R21.1, R24.2, R25.2
- net MIDI_IN: now also R2.1; no longer R22.1
- net N$12: now also R10.2; no longer R15.2
- net N$15: now also R12.2; no longer R13.2
- net N$16: now also R4.2; no longer R23.2
- net N$18: now also R4.1; no longer R23.1
- net N$20: now also R14.2; no longer R11.2
- net N$21: now also D2.A; no longer D3.A
- net N$24: now also R11.2; no longer R16.2
- net N$28: now also R6.1; no longer R24.1
- net N$33: now also R13.2; no longer R14.2
- net N$35: now also R15.2; no longer R12.2
- net N$36: now also R17.2; no longer R10.2
- net N$37: now also R19.2; no longer R8.2
- net N$38: now also R21.2; no longer R3.2
- net N$4: now also R3.2; no longer R21.2
- net N$5: now also R5.1; no longer R25.1
- net N$57: now also R16.2; no longer R2.2
- net N$6: now also R7.2; no longer R20.2
- net N$60: now also R18.2; no longer R4.2
- net N$63: now also R20.2; no longer R5.2
- net N$66: now also R22.2; no longer R6.2
- net N$7: now also R9.2; no longer R18.2
- net N$8: now also D3.P$1; no longer U$10.P$1
- net N$9: now also R8.2; no longer R17.2
- net OUT1: now also R7.1, R8.1; no longer R17.1, R20.1
- net OUT2: now also R10.1, R9.1; no longer R15.1, R18.1
- net OUT3: now also R11.1, R12.1; no longer R13.1, R16.1
- net OUT4: now also R13.1; no longer R11.1
- net OUT5: now also R15.1, R16.1; no longer R12.1, R2.1
- net OUT6: now also R17.1, R18.1; no longer R10.1, R4.1
- net OUT7: now also R19.1, R20.1; no longer R5.1, R8.1
- net OUT8: now also R21.1, R22.1; no longer R3.1, R6.1
Other:
- moved on the sheet: R10, R11, R12, R13, R14, R15, R16, R17, R18, R2, R20, R21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
