File: relay_sw_ssr/ssr_board.brd (EAGLE design)
At the start: 34.5 x 44.2 mm, 40 parts, among them IC1 PIC16F1825SO14, IC2 6N138

Commit message: ssr switcher v1
Parts:
- removed U1: (no value), microbuilder:SOT223-W
- added IC3: 6N138, optocoupler:DIL08
- C1: device rcl:E2-5 -> rcl:C0805
- C4: device rcl:C0805 -> rcl:E2-5
- IC2: value 6N138 -> (none); device optocoupler:DIL08 -> microbuilder:SOT223-W
- R1: value 1k -> 100r
- R10: value 1k5 -> 1k
- R9: value 100r -> 1k5
- moved C1 29.3 mm to (29.2, 77.5), turned to 180 degrees
- moved R10 26.3 mm to (41.8, 75.4), turned to 270 degrees
- moved R1 19.0 mm to (22.9, 77.5), turned to 0 degrees
- moved C2 17.6 mm to (38.0, 62.2), turned to 0 degrees
- moved IC2 15.7 mm to (45.7, 62.2), flipped to the top, turned to 270 degrees
- moved C4 12.2 mm to (47.5, 54.6), flipped to the bottom, turned to 180 degrees
- moved R3 2.54 mm to (22.9, 72.4), turned to 0 degrees
- moved R4 2.54 mm to (22.9, 69.8), turned to 180 degrees
- moved R6 2.54 mm to (22.9, 64.8), turned to 180 degrees
- moved R7 2.54 mm to (22.9, 62.2), turned to 0 degrees
- moved R8 2.54 mm to (22.9, 59.7), turned to 180 degrees
- moved R9 2.54 mm to (22.9, 57.1), turned to 0 degrees
- moved R2 2.54 mm to (22.9, 74.9), turned to 180 degrees
- moved R5 2.54 mm to (22.9, 67.3), turned to 0 degrees
- flipped C5 to the bottom, turned to 180 degrees
- renumbered D4 to D2, D5 to D1, J1 to ICSP, U$1 to D3
Connections:
- net 5V: now also C1.1, IC3.8, R10.1; no longer C2.1, IC2.8, R1.1
- net GND: now also C1.2, C2.1, C4.-, IC2.1, IC3.5, R9.1; no longer C1.-, C2.2, C4.1, IC2.5, R10.1, U1.1
- net N$10: now also IC3.2; no longer IC2.2
- net N$11: now also IC3.3; no longer IC2.3
- net N$12: now also IC3.7, R9.2; no longer IC2.7, R10.2
- net N$14: now also R3.1; no longer R4.1
- net N$15: now also R2.2; no longer R3.2
- net N$16: now also R1.1; no longer R2.1
- net N$17: now also R6.2; no longer R7.2
- net N$18: now also R8.2; no longer R9.2
- net N$19: now also R5.1; no longer R6.1
- net N$2: now also C2.2, IC2.2; no longer C4.2, U1.2
- net N$20: now also R7.1; no longer R8.1
- net N$21: now also R2.1; no longer R3.1
- net N$22: now also R1.2; no longer R2.2
- net N$23: now also R6.1; no longer R7.1
- net N$24: now also R8.1; no longer R9.1
- net N$25: now also R5.2; no longer R6.2
- net N$26: now also R7.2; no longer R8.2
- net N$27: now also R4.2; no longer R5.2
- net N$4: now also R10.2; no longer R1.2
- net N$46: now also R3.2; no longer R4.2
- net N$47: now also R4.1; no longer R5.1
- net N$48: now also IC3.6; no longer IC2.6
- net N$5: now also C4.+, IC2.3; no longer C1.+, U1.3
Routing:
- net N$12: track 18.0 -> 16.0 mm
- net N$21: track 11.8 -> 12.9 mm
- net N$5: track 11.2 -> 12.1 mm
- net N$46: track 14.1 -> 13.6 mm
- net GND: vias 1 -> 3
Other:
- board text added: "CH1"
- board text added: "CH2"
- board text added: "CH3"
- board text added: "CH4"
- board text added: "CH5"
- board text added: "CH6"
- board text added: "CH7"
- board text added: "CH8"
- board text added: "DC+"
- board text added: "DC-"
- board text added: "SSR MIDI SWITCHER v1"
- board text added: "six4pix.com"
