File: relay_sw_ssr/ssr_board.sch (EAGLE design)
At the start: 40 parts, among them IC1 PIC16F1825SO14, IC2 6N138

Commit message: ssr switcher v1
Parts:
- removed U1: (no value), microbuilder:LM1117SOT223-WAVE
- added IC3: 6N138, optocoupler:6N138
- C1: device rcl:CPOL-EUE2-5 -> rcl:C-EUC0805
- C4: device rcl:C-EUC0805 -> rcl:CPOL-EUE2-5
- IC2: value 6N138 -> (none); device optocoupler:6N138 -> microbuilder:LM1117SOT223-WAVE
- R1: value 1k -> 100r
- R10: value 1k5 -> 1k
- R9: value 100r -> 1k5
- renumbered D4 to D2, D5 to D1, J1 to ICSP, U$1 to D3
Connections:
- net 5V: now also C1.1, IC3.VCC, R10.1; no longer C2.1, IC2.VCC, R1.1
- net GND: now also C1.2, C2.1, C4.-, IC2.ADJ, IC3.GND, R9.1; no longer C1.-, C2.2, C4.1, IC2.GND, R10.1, U1.ADJ
- net N$10: now also IC3.A; no longer IC2.A
- net N$11: now also IC3.C; no longer IC2.C
- net N$12: now also IC3.VB, R9.2; no longer IC2.VB, R10.2
- net N$14: now also R3.1; no longer R4.1
- net N$15: now also R2.2; no longer R3.2
- net N$16: now also R1.1; no longer R2.1
- net N$17: now also R6.2; no longer R7.2
- net N$18: now also R8.2; no longer R9.2
- net N$19: now also R5.1; no longer R6.1
- net N$2: now also C2.2, IC2.OUT; no longer C4.2, U1.OUT
- net N$20: now also R7.1; no longer R8.1
- net N$21: now also R2.1; no longer R3.1
- net N$22: now also R1.2; no longer R2.2
- net N$23: now also R6.1; no longer R7.1
- net N$24: now also R8.1; no longer R9.1
- net N$25: now also R5.2; no longer R6.2
- net N$26: now also R7.2; no longer R8.2
- net N$27: now also R4.2; no longer R5.2
- net N$4: now also R10.2; no longer R1.2
- net N$46: now also R3.2; no longer R4.2
- net N$47: now also R4.1; no longer R5.1
- net N$48: now also IC3.VO; no longer IC2.VO
- net N$5: now also C4.+, IC2.IN; no longer C1.+, U1.IN
Other:
- moved on the sheet: C2, R1, R10, R2, R3, R4, R5, R6, R7, R8, R9
