File: midi_switcher_smt/midi-switcher-smt.sch (EAGLE design)
At the start: 79 parts, among them IC1 6N138, IC2 PIC16F1825SO14, IC3 LD1086, Q1 MJD122GDPAK, Q2 MJD122GDPAK, Q3 MJD122GDPAK, Q4 MJD122GDPAK, Q5 MJD122GDPAK, Q6 MJD122GDPAK, Q7 MJD122GDPAK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

Commit message: Rev 3B board (single) enlarge terminal pin holes
Parts:
- OP1+, OP1-, OP2+, OP2-, OP3+, OP3-, OP4+, OP4-, OP5+, OP5-, OP6-, OP7+, OP7-, OP8+, OP8+1, OP8-, POWER+1, POWER+2, POWER-1, POWER-2: device adafruit:PINHD-1X1 -> jason_eagle6:PINHD-1X1
Changed lines of the file:
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@@
 <layer number="56" name="wert" color="7" fill="1" visible="no" active="no"/>
 <layer number="57" name="tCAD" color="7" fill="1" visible="no" active="no"/>
+<layer number="90" name="Modules" color="7" fill="1" visible="yes" active="yes"/>
 <layer number="91" name="Nets" color="2" fill="1" visible="yes" active="yes"/>
 <layer number="92" name="Busses" color="1" fill="1" visible="yes" active="yes"/>
@@
 <part name="R2" library="rcl" deviceset="R-EU_" device="R0805"/>
 <part name="ICSP" library="microbuilder" deviceset="HEADER-1X6" device=""/>
-<part name="OP1-" library="adafruit" deviceset="PINHD-1X1" device=""/>
-<part name="OP2-" library="adafruit" deviceset="PINHD-1X1" device=""/>
-<part name="OP3-" library="adafruit" deviceset="PINHD-1X1" device=""/>
-<part name="OP4-" library="adafruit" deviceset="PINHD-1X1" device=""/>
-<part name="OP5-" library="adafruit" deviceset="PINHD-1X1" device=""/>
-<part name="OP6-" library="adafruit" deviceset="PINHD-1X1" device=""/>
-<part name="OP7-" library="adafruit" deviceset="PINHD-1X1" device=""/>
-<part name="OP8-" library="adafruit" deviceset="PINHD-1X1" device=""/>
-<part name="OP1+" library="adafruit" deviceset="PINHD-1X1" device=""/>
-<part name="OP2+" library="adafruit" deviceset="PINHD-1X1" device=""/>
-<part name="OP3+" library="adafruit" deviceset="PINHD-1X1" device=""/>
-<part name="OP4+" library="adafruit" deviceset="PINHD-1X1" device=""/>
-<part name="OP5+" library="adafruit" deviceset="PINHD-1X1" device=""/>
-<part name="OP7+" library="adafruit" deviceset="PINHD-1X1" device=""/>
-<part name="OP8+" library="adafruit" deviceset="PINHD-1X1" device=""/>
+<part name="OP1-" library="jason_eagle6" deviceset="PINHD-1X1" device=""/>
+<part name="OP2-" library="jason_eagle6" deviceset="PINHD-1X1" device=""/>
+<part name="OP3-" library="jason_eagle6" deviceset="PINHD-1X1" device=""/>
+<part name="OP4-" library="jason_eagle6" deviceset="PINHD-1X1" device=""/>
+<part name="OP5-" library="jason_eagle6" deviceset="PINHD-1X1" device=""/>
+<part name="OP6-" library="jason_eagle6" deviceset="PINHD-1X1" device=""/>
+<part name="OP7-" library="jason_eagle6" deviceset="PINHD-1X1" device=""/>
+<part name="OP8-" library="jason_eagle6" deviceset="PINHD-1X1" device=""/>
+<part name="OP1+" library="jason_eagle6" deviceset="PINHD-1X1" device=""/>
+<part name="OP2+" library="jason_eagle6" deviceset="PINHD-1X1" device=""/>
+<part name="OP3+" library="jason_eagle6" deviceset="PINHD-1X1" device=""/>
+<part name="OP4+" library="jason_eagle6" deviceset="PINHD-1X1" device=""/>
+<part name="OP5+" library="jason_eagle6" deviceset="PINHD-1X1" device=""/>
+<part name="OP7+" library="jason_eagle6" deviceset="PINHD-1X1" device=""/>
+<part name="OP8+" library="jason_eagle6" deviceset="PINHD-1X1" device=""/>
 <part name="C1" library="rcl" deviceset="C-EU" device="C0805"/>
 <part name="C3" library="rcl" deviceset="C-EU" device="C0805"/>
@@
 <part name="C4" library="rcl" deviceset="CPOL-EU" device="E2.5-7"/>
 <part name="D3" library="jasons_stuff" deviceset="1N4004" device=""/>
-<part name="POWER+1" library="adafruit" deviceset="PINHD-1X1" device=""/>
-<part name="POWER+2" library="adafruit" deviceset="PINHD-1X1" device=""/>
-<part name="POWER-1" library="adafruit" deviceset="PINHD-1X1" device=""/>
-<part name="POWER-2" library="adafruit" deviceset="PINHD-1X1" device=""/>
+<part name="POWER+1" library="jason_eagle6" deviceset="PINHD-1X1" device=""/>
+<part name="POWER+2" library="jason_eagle6" deviceset="PINHD-1X1" device=""/>
+<part name="POWER-1" library="jason_eagle6" deviceset="PINHD-1X1" device=""/>
+<part name="POWER-2" library="jason_eagle6" deviceset="PINHD-1X1" device=""/>
 <part name="U$1" library="adafruit" deviceset="2.1MMJACK" device="THM"/>
 <part name="D2" library="jasons_stuff" deviceset="1N4004" device=""/>
@@
 <part name="GND17" library="supply1" deviceset="GND" device=""/>
 <part name="GND18" library="supply1" deviceset="GND" device=""/>
-<part name="OP8+1" library="adafruit" deviceset="PINHD-1X1" device=""/>
+<part name="OP8+1" library="jason_eagle6" deviceset="PINHD-1X1" device=""/>
 </parts>
 <sheets>
